Commit message: Mapping is done, navigating to the aruco codes is resulting in some issues, will need to check with Motaz to see if he knows a fix

File: src/final_project/urdf/turtlebot3_burger.xacro (robot description, xacro)
@@ -6,5 +6,5 @@
   <xacro:property name="namespace" value="$(arg namespace)"/>
   <!-- <xacro:property name="mesh_path" value="package://homework3/meshes"/> -->
-  <xacro:property name="mesh_path" value="file://$(find vision_demo)/meshes"/>
+  <xacro:property name="mesh_path" value="file://$(find final_project)/meshes"/>
   <!-- <xacro:property name="mesh_path" value="file:///home/sean/ros2_course_ws_master/install/homework3/share/homework3/meshes"/> -->
   <!-- Init colour -->
